Commit message: initial commit

File: src/jackal_description/urdf/accessories.urdf.xacro (robot description, xacro)
@@ -23,6 +23,6 @@
   <xacro:include filename="$(find jackal_description)/urdf/accessories/hdl32_mount.urdf.xacro" />
   <!--
-    Add Microstrain IMU. By default the Jackal comes equipped with an IMU linked to "imu_link". These extra
-    optional microstrain IMU's will be added to another frame, by default, "microstrain_link".
+    Add Microstrain IMU. By default the Jackal comes equipped with an IMU linked to "imu_link".
+    These extra optional microstrain IMU's will be added to another frame, by default, "microstrain_link".
   -->
   <xacro:if value="$(optenv JACKAL_IMU_MICROSTRAIN 0)">
@@ -39,6 +39,6 @@
   </xacro:if>
   <!--
-    Add primary/secondary 2D lidar sensors.  By default these are SICK LMS1xx but can be changed with the
-    JACKAL_LASER_MODEL and JACKAL_LASER_SECONDARY_MODEL environment variables. Valid model designations are:
+    Add primary/secondary 2D lidar sensors.
+    By default these are SICK LMS1xx but can be changed with JACKAL_LASER_MODEL, etc.
     - lms1xx (default) :: SICK LMS1xx
     - ust10            :: Hokuyo UST10
@@ -74,5 +74,5 @@
         <link name="${prefix}_laser_base"/>
         <joint name="${prefix}_laser_base_joint" type="fixed">
-          <origin xyz="$(optenv JACKAL_LASER_OFFSET 0 0 0)" rpy="$(optenv JACKAL_LASER_RPY 0 0 0)"/>
+          <origin xyz="$(optenv JACKAL_LASER_OFFSET 0 0 0)" rpy="$(optenv JACKAL_LASER_RPY 0 0 0)" />
           <parent link="${parent}"/>
           <child link="${prefix}_laser_base"/>
@@ -85,5 +85,5 @@
       </xacro:unless>
     </xacro:if>
-    <!-- SICK Tim -->
+    <!-- SICK Tim (tim551) -->
     <xacro:if value="${lidar_model == 'tim551'}">
       <xacro:property name="prefix" value="$(optenv JACKAL_LASER_PREFIX tim551)" />
@@ -164,5 +164,5 @@
   </xacro:if>
   <!--
-    Add a 3D lidar sensor.  By default this is a Velodyne VLP16 but can be changed with the
+    Add a 3D lidar sensor. Default is Velodyne VLP16, can set JACKAL_LASER_3D_MODEL=hdl32e etc.
     JACKAL_LASER_3D_MODEL environment variable. Valid model designations are:
     - vlp16 (default)  :: Velodyne VLP16
@@ -203,5 +203,5 @@
     <xacro:property name="parent" value="$(optenv JACKAL_NAVSAT_PARENT ${mount}_mount)" />
     <xacro:property name="navsat_model" value="$(optenv JACKAL_NAVSAT_MODEL smart6)" />
-    <!--- Novotel Smart6 -->
+    <!-- Novatel Smart6 -->
     <xacro:if value="${navsat_model == 'smart6'}">
       <xacro:novatel_smart6 prefix="${prefix}"/>
@@ -226,5 +226,5 @@
       </xacro:unless>
     </xacro:if>
-    <!-- Novotel Smart7 -->
+    <!-- Novatel Smart7 -->
     <xacro:if value="${navsat_model == 'smart7'}">
       <xacro:novatel_smart7 prefix="${prefix}"/>
@@ -250,14 +250,8 @@
     </xacro:if>
   </xacro:if>
-  <!--
-    Add Cameras.
-    - JACKAL_FLEA3
-    - JACKAL_STEREO_FLEA3
-    - JACKAL_BB2
-  -->
   <!-- Common camera mounts and accessory URDFs. -->
   <xacro:include filename="$(find jackal_description)/urdf/accessories/camera_mount.urdf.xacro" />
   <xacro:include filename="$(find pointgrey_camera_description)/urdf/pointgrey_flea3.urdf.xacro" />
-  <!-- If enabled, generate the flea3 camera payload with a tilt of 30 degrees. -->
+  <!-- 如果启用的话，生成前方的PointGrey Flea3相机（默认朝前），示例保留 -->
   <xacro:if value="$(optenv JACKAL_FLEA3 1)">
     <xacro:property name="name" value="$(optenv JACKAL_FLEA3_NAME front)" />
@@ -269,6 +263,6 @@
     <xacro:pointgrey_flea3 frame="${prefix}_camera" name="${name}"
       camera_x="0.0754" camera_y="0.029" camera_z="0.029"
-      camera_mass="0.085" hfov="1.0471975512" fps="60" width="640" height="512"/>
-    <!-- Mount Enabled -->
+      camera_mass="0.085" hfov="1.0471975512" fps="60" width="2560" height="1440"/>
+    <!-- 有挂架 -->
     <xacro:if value="${tower}">
       <xacro:camera_mount prefix="${prefix}" tilt="${tilt}"/>
@@ -285,5 +279,5 @@
       </joint>
     </xacro:if>
-    <!-- Mount Disabled -->
+    <!-- 无挂架 -->
     <xacro:unless value="${tower}">
       <link name="${prefix}_camera_base"/>
@@ -295,6 +289,5 @@
       </joint>
       <joint name="${prefix}_camera_joint" type="fixed">
-        <origin xyz="0 0 0.0145"
-                rpy="0 0 0" />
+        <origin xyz="0 0 0.0145" rpy="0 0 0" />
         <parent link="${prefix}_camera_base" />
         <child link="${prefix}_camera" />
@@ -303,6 +296,5 @@
   </xacro:if>
   <xacro:include filename="$(find jackal_description)/urdf/accessories/stereo_camera_mount.urdf.xacro" />
-  <!-- If enabled, generates a pair of flea3 cameras for stereo vision with a tilt of 30 degrees. -->
-  <!-- Disabled temporarily due to metapackage issue. -->
+  <!-- 如果启用的话，生成一对 Flea3 立体相机（默认朝前），示例保留 -->
   <xacro:if value="$(optenv JACKAL_STEREO_FLEA3 0)">
     <xacro:property name="tilt" value="$(optenv JACKAL_FLEA3_TILT 0.5236)"/>
@@ -337,8 +329,6 @@
     </joint>
   </xacro:if>
-  <!-- If enabled, generate the bumblebee2 camera payload with a tilt of 0 degrees. -->
+  <!-- Bumblebee2 camera -->
   <xacro:include filename="$(find pointgrey_camera_description)/urdf/pointgrey_bumblebee2.urdf.xacro" />
-  <!-- If enabled, generate the bumblebee2 camera payload with a tilt of 0 degrees. -->
-  <!-- Disabled temporarily due to metapackage issue. -->
   <xacro:if value="$(optenv JACKAL_BB2 0)">
     <xacro:property name="tilt" value="$(optenv JACKAL_BB2_TILT 0)" />
@@ -380,5 +370,5 @@
     </xacro:unless>
   </xacro:if>
-  <!-- BlackflyS Camera -->
+  <!-- BlackflyS camera -->
   <xacro:include filename="$(find flir_camera_description)/urdf/flir_blackflys.urdf.xacro"/>
   <xacro:if value="$(optenv JACKAL_BLACKFLY 0)">
@@ -461,3 +451,148 @@
     </gazebo>
   </xacro:if>
+  <!-- ============= 左侧摄像头（朝向左侧） ============= -->
+  <xacro:if value="$(optenv JACKAL_LEFT_CAMERA 1)">
+    <!-- 定义相关参数 -->
+    <xacro:property name="name" value="$(optenv JACKAL_LEFT_CAMERA_NAME left_camera)" />
+    <xacro:property name="tilt" value="$(optenv JACKAL_LEFT_CAMERA_TILT 0.)" />
+    <xacro:property name="tower" value="$(optenv JACKAL_LEFT_CAMERA_TOWER 1)" />
+    <xacro:property name="mount" value="$(optenv JACKAL_LEFT_CAMERA_MOUNT left)" />
+    <xacro:property name="prefix" value="$(optenv JACKAL_LEFT_CAMERA_PREFIX ${mount})" />
+    <!-- 缺省：父链接 = left_mount -->
+    <xacro:property name="parent" value="$(optenv JACKAL_LEFT_CAMERA_PARENT ${mount}_mount)" />
+    <!-- 利用 pointgrey_flea3 定义摄像头外观和参数 (也可换成其它摄像头) -->
+    <xacro:pointgrey_flea3 frame="${prefix}_camera" name="${name}"
+        camera_x="0.0754" camera_y="0.029" camera_z="0.029"
+        camera_mass="0.085" hfov="1.0471975512" fps="60" width="2560" height="1440"/>
+    <!-- 如果有塔架 (tower=1) -->
+    <xacro:if value="${tower}">
+      <xacro:camera_mount prefix="${prefix}" tilt="${tilt}"/>
+      <joint name="${prefix}_camera_mount_joint" type="fixed">
+        <!--
+          xyz: 将摄像头相对于 left_mount 的位置做一个偏移
+          rpy: 让摄像头光轴朝向左方(绕Z转+90°=1.5708 rad)
+        -->
+        <origin xyz="$(optenv JACKAL_LEFT_CAMERA_OFFSET 0 0.0 0.3)"
+                rpy="$(optenv JACKAL_LEFT_CAMERA_RPY 0 0 1.5708)" />
+        <parent link="${parent}" />
+        <child link="${prefix}_camera_mount" />
+      </joint>
+      <joint name="${prefix}_camera_bracket_joint" type="fixed">
+        <origin xyz="0.020 0 0.0245" rpy="0 0 0" />
+        <parent link="${prefix}_camera_beam" />
+        <child link="${prefix}_camera" />
+      </joint>
+    </xacro:if>
+    <!-- 如果tower=0，不需要相机支架，也让相机面向左方 -->
+    <xacro:unless value="${tower}">
+      <link name="${prefix}_camera_base"/>
+      <joint name="${prefix}_camera_base_joint" type="fixed">
+        <origin xyz="$(optenv JACKAL_LEFT_CAMERA_OFFSET 0 0.0 5)"
+                rpy="$(optenv JACKAL_LEFT_CAMERA_RPY 0 0.5 1.5708)" />
+        <parent link="${parent}" />
+        <child link="${prefix}_camera_base" />
+      </joint>
+      <joint name="${prefix}_camera_joint" type="fixed">
+        <origin xyz="0 0 0.0145" rpy="0 0 0" />
+        <parent link="${prefix}_camera_base" />
+        <child link="${prefix}_camera" />
+      </joint>
+    </xacro:unless>
+    <!-- 在 Gazebo 中生成摄像头插件，发布图像话题 -->
+    <gazebo reference="${prefix}_camera">
+      <sensor type="camera" name="${name}_sensor">
+        <update_rate>30</update_rate>
+        <camera>
+          <horizontal_fov>1.0471975512</horizontal_fov>
+          <image>
+            <width>2560</width>
+            <height>1440</height>
+            <format>R8G8B8</format>
+          </image>
+          <clip>
+            <near>0.1</near>
+            <far>100</far>
+          </clip>
+        </camera>
+        <plugin name="gazebo_ros_camera_controller" filename="libgazebo_ros_camera.so">
+          <robotNamespace>/left_camera</robotNamespace>
+          <cameraName>${name}_sensor</cameraName>
+          <imageTopicName>image_raw</imageTopicName>
+          <cameraInfoTopicName>camera_info</cameraInfoTopicName>
+        </plugin>
+      </sensor>
+    </gazebo>
+  </xacro:if>
+  <!-- =========== 左侧摄像头定义到此结束 =========== -->
+  <!-- ============= 第二个左侧摄像头（俯角不同） ============= -->
+  <xacro:if value="$(optenv JACKAL_LEFT_CAMERA2 1)">
+    <!-- 定义相关参数，除俯角外其他与原左侧相机相同 -->
+    <xacro:property name="name" value="$(optenv JACKAL_LEFT_CAMERA2_NAME left_camera_2)" />
+    <!-- 此处默认俯角设置为 0.1 rad，可通过环境变量 JACKAL_LEFT_CAMERA2_TILT 覆盖 -->
+    <xacro:property name="tilt" value="$(optenv JACKAL_LEFT_CAMERA2_TILT 0.1)" />
+    <xacro:property name="tower" value="$(optenv JACKAL_LEFT_CAMERA2_TOWER 1)" />
+    <xacro:property name="mount" value="$(optenv JACKAL_LEFT_CAMERA2_MOUNT left)" />
+    <!-- 修改：第二个左侧摄像头默认父链接改为 left_mount_2 -->
+    <xacro:property name="parent" value="$(optenv JACKAL_LEFT_CAMERA2_PARENT left_mount_2)" />
+    <!-- 修改前缀，确保链接名不重复，默认设置为 "left_2" -->
+    <xacro:property name="prefix" value="$(optenv JACKAL_LEFT_CAMERA2_PREFIX ${mount}_2)" />
+    <!-- 利用 pointgrey_flea3 定义摄像头外观和参数 -->
+    <xacro:pointgrey_flea3 frame="${prefix}_camera" name="${name}"
+        camera_x="0.0754" camera_y="0.029" camera_z="0.029"
+        camera_mass="0.085" hfov="1.0471975512" fps="60" width="2560" height="1440"/>
+    <!-- 如果有塔架 (tower=1) -->
+    <xacro:if value="${tower}">
+      <xacro:camera_mount prefix="${prefix}" tilt="${tilt}"/>
+      <joint name="${prefix}_camera_mount_joint" type="fixed">
+        <origin xyz="$(optenv JACKAL_LEFT_CAMERA2_OFFSET 0 0.0 0.3)"
+                rpy="$(optenv JACKAL_LEFT_CAMERA2_RPY 0 0 1.5708)" />
+        <parent link="${parent}" />
+        <child link="${prefix}_camera_mount" />
+      </joint>
+      <joint name="${prefix}_camera_bracket_joint" type="fixed">
+        <origin xyz="0.020 0 0.0245" rpy="0 0 0" />
+        <parent link="${prefix}_camera_beam" />
+        <child link="${prefix}_camera" />
+      </joint>
+    </xacro:if>
+    <!-- 如果 tower=0 -->
+    <xacro:unless value="${tower}">
+      <link name="${prefix}_camera_base"/>
+      <joint name="${prefix}_camera_base_joint" type="fixed">
+        <origin xyz="$(optenv JACKAL_LEFT_CAMERA2_OFFSET 0 0.0 5)"
+                rpy="$(optenv JACKAL_LEFT_CAMERA2_RPY 0 0.5 1.5708)" />
+        <parent link="${parent}" />
+        <child link="${prefix}_camera_base" />
+      </joint>
+      <joint name="${prefix}_camera_joint" type="fixed">
+        <origin xyz="0 0 0.0145" rpy="0 0 0" />
+        <parent link="${prefix}_camera_base" />
+        <child link="${prefix}_camera" />
+      </joint>
+    </xacro:unless>
+    <!-- 在 Gazebo 中生成摄像头插件 -->
+    <gazebo reference="${prefix}_camera">
+      <sensor type="camera" name="${name}_sensor">
+        <update_rate>30</update_rate>
+        <camera>
+          <horizontal_fov>1.0471975512</horizontal_fov>
+          <image>
+            <width>2560</width>
+            <height>1440</height>
+            <format>R8G8B8</format>
+          </image>
+          <clip>
+            <near>0.1</near>
+            <far>100</far>
+          </clip>
+        </camera>
+        <plugin name="gazebo_ros_camera_controller" filename="libgazebo_ros_camera.so">
+          <robotNamespace>/left_camera_2</robotNamespace>
+          <cameraName>${name}_sensor</cameraName>
+          <imageTopicName>image_raw</imageTopicName>
+          <cameraInfoTopicName>camera_info</cameraInfoTopicName>
+        </plugin>
+      </sensor>
+    </gazebo>
+  </xacro:if>
 </robot>

File: src/jackal_description/urdf/jackal.urdf.xacro (robot description, xacro)
@@ -80,5 +80,5 @@
     <origin xyz="${-wheelbase/2} ${-track/2} ${wheel_vertical_offset}" rpy="0 0 0" />
   </xacro:wheel>
-  <link name="base_link"></link>
+  <link name="base_link" />
   <joint name="base_link_joint" type="fixed">
     <origin xyz="0 0 0" rpy="0 0 0" />
@@ -104,10 +104,10 @@
       <origin xyz="0.012  0.002 0.067" rpy="0 0 0"/>
       <mass value="16.523"/>
-      <!-- Moments of inertia: ( chassis without wheels ) -->
+      <!-- Moments of inertia -->
       <inertia
         ixx="0.3136" ixy="-0.0008" ixz="0.0164"
         iyy="0.3922" iyz="-0.0009"
         izz="0.4485"/>
-      </inertial>
+    </inertial>
   </link>
   <xacro:unless value="$(optenv JACKAL_FRONT_ACCESSORY_FENDER 0)">
@@ -200,5 +200,5 @@
     <origin xyz="-0.180 0.126 0.1815" />
   </joint>
-  <link name="mid_mount"></link>
+  <link name="mid_mount" />
   <joint name="mid_mount_joint" type="fixed">
     <parent link="chassis_link" />
@@ -206,5 +206,5 @@
     <origin xyz="0 0 ${chassis_height}" />
   </joint>
-  <link name="rear_mount"></link>
+  <link name="rear_mount" />
   <joint name="rear_mount_joint" type="fixed">
     <parent link="mid_mount" />
@@ -212,5 +212,5 @@
     <origin xyz="${-mount_spacing} 0 0" />
   </joint>
-  <link name="front_mount"></link>
+  <link name="front_mount" />
   <joint name="front_mount_joint" type="fixed">
     <parent link="mid_mount" />
@@ -218,5 +218,22 @@
     <origin xyz="${mount_spacing} 0 0" />
   </joint>
-  <!-- Bring in simulation data for Gazebo. -->
+  <!-- 左侧挂载点 link -->
+  <link name="left_mount"/>
+  <!-- 将 left_mount 固定到 mid_mount 上 -->
+  <joint name="left_mount_joint" type="fixed">
+    <parent link="mid_mount" />
+    <child link="left_mount" />
+    <!-- 沿 Y 方向偏移 mount_spacing 到左侧，并与 mid_mount 同样的高度 -->
+    <origin xyz="0 0.12 4" rpy="-0.42 0 0"/>
+  </joint>
+  <!-- 新增：第二个左侧挂载点定义，必须在加载 accessories.urdf.xacro 前定义 -->
+  <link name="left_mount_2"/>
+  <joint name="left_mount_2_joint" type="fixed">
+    <parent link="left_mount" />
+    <child link="left_mount_2" />
+    <!-- 根据需要设置一个轻微偏移（例如沿 X 方向偏移 0.1 m） -->
+    <origin xyz="0.1 0 0" rpy="-0.275 0 0"/>
+  </joint>
+ <!-- Bring in simulation data for Gazebo. -->
   <xacro:include filename="$(find jackal_description)/urdf/jackal.gazebo" />
   <!-- Optional standard accessories, including their simulation data. The rendering
@@ -224,7 +241,3 @@
        default each one to off.-->
   <xacro:include filename="$(find jackal_description)/urdf/accessories.urdf.xacro" />
-  <!-- Optional custom includes. -->
-  <xacro:include filename="$(optenv JACKAL_URDF_EXTRAS empty.urdf)" />
-  <!-- Optional for Clearpath internal softwares -->
-  <xacro:include filename="$(optenv CPR_URDF_EXTRAS empty.urdf)" />
 </robot>
